Commit message: Add modifications after RViz Integration part for project GoChaseIt

File: catkin_ws/src/my_robot/urdf/my_robot.xacro (robot description, xacro)
@@ -1,4 +1,5 @@
 <?xml version='1.0'?>
 <robot name="my_robot" xmlns:xacro="http://www.ros.org/wiki/xacro">
+  <xacro:include filename="$(find my_robot)/urdf/my_robot.gazebo" />
   <link name="robot_footprint"></link>
   <joint name="robot_footprint_joint" type="fixed">
@@ -65,5 +66,5 @@
       />
     </inertial>
-    <collision name='collision'>
+    <collision name='left_wheel_collision'>
       <origin xyz="0 0 0" rpy=" 0 1.507 1.507"/>
       <geometry>
@@ -71,5 +72,5 @@
       </geometry>
     </collision>
-    <visual name='chassis_visual'>
+    <visual name='left_wheel_visual'>
       <origin xyz="0 0 0" rpy=" 0 1.507 1.507"/>
       <geometry>
@@ -88,5 +89,5 @@
       />
     </inertial>
-    <collision name='collision'>
+    <collision name='right_wheel_collision'>
       <origin xyz="0 0 0" rpy=" 0 1.507 1.507"/>
       <geometry>
@@ -94,5 +95,5 @@
       </geometry>
     </collision>
-    <visual name='chassis_visual'>
+    <visual name='right_wheel_visual'>
       <origin xyz="0 0 0" rpy=" 0 1.507 1.507"/>
       <geometry>
@@ -117,3 +118,73 @@
     <dynamics damping="1.0" friction="1.0"/>
   </joint>
+	<link name='camera'>
+		<inertial>
+      <mass value="0.1"/>
+      <origin xyz="0.0 0 0" rpy=" 0 0 0"/>
+      <inertia
+          ixx="0.000001" ixy="0" ixz="0"
+          iyy="0.000001" iyz="0"
+          izz="0.000001"
+      />
+    </inertial>
+    <collision name='camera_collision'>
+      <origin xyz="0 0 0" rpy=" 0 0 0"/>
+      <geometry>
+        <box size="0.05 0.05 0.05"/>
+      </geometry>
+    </collision>
+    <visual name='camera_visual'>
+      <origin xyz="0 0 0" rpy=" 0 0 0"/>
+      <geometry>
+        <box size="0.05 0.05 0.05"/>
+      </geometry>
+    </visual>
+	</link>
+	<joint type="fixed" name="camera_joint">
+    <origin xyz="0.2 0 0" rpy="0 0 0"/>
+    <child link="camera"/>
+    <parent link="chassis"/>
+    <axis xyz="0 1 0" rpy="0 0 0"/>
+  </joint>
+	<link name='hokuyo'>
+		<inertial>
+      <mass value="0.00001"/>
+      <origin xyz="0 0 0" rpy=" 0 0 0"/>
+      <inertia
+          ixx="0.000001" ixy="0" ixz="0"
+          iyy="0.000001" iyz="0"
+          izz="0.000001"
+      />
+    </inertial>
+    <collision name='hokuyo_collision'>
+      <origin xyz="0 0 0" rpy=" 0 0 0"/>
+      <geometry>
+        <box size='0.1 0.1 0.1'/>
+      </geometry>
+    </collision>
+    <visual name='hokuyo_visual'>
+      <origin xyz="0 0 0" rpy=" 0 0 0"/>
+      <geometry>
+				<mesh filename = 'package://my_robot/meshes/hokuyo.dae'/>
+			</geometry>
+    </visual>
+	</link>
+	<joint type="fixed" name="hokuyo_joint">
+    <origin xyz="0.15 0 0.1" rpy="0 0 0"/>
+    <child link="hokuyo"/>
+    <parent link="chassis"/>
+    <axis xyz="0 1 0" rpy="0 0 0"/>
+  </joint>
+	<gazebo reference="left_wheel">
+    <material>Gazebo/Green</material>
+	</gazebo>
+	<gazebo reference="right_wheel">
+    <material>Gazebo/Green</material>
+	</gazebo>
+	<gazebo reference="chassis">
+    <material>Gazebo/Blue</material>
+	</gazebo>
+	<gazebo reference="camera">
+    <material>Gazebo/Red</material>
+	</gazebo>
 </robot>
