Commit message: Changed the robot to a 6 wheels one

File: Project 2/my_robot/urdf/my_robot.xacro (robot description, xacro)
@@ -69,5 +69,5 @@
       <origin xyz="0 0 0" rpy=" 0 1.507 1.507"/>
       <geometry>
-        <cylinder length='0.05' radius='0.1'/>
+        <cylinder length='0.05' radius='0.05'/>
       </geometry>
     </collision>
@@ -75,5 +75,5 @@
       <origin xyz="0 0 0" rpy=" 0 1.507 1.507"/>
       <geometry>
-        <cylinder length='0.05' radius='0.1'/>
+        <cylinder length='0.05' radius='0.05'/>
       </geometry>
     </visual>
@@ -92,5 +92,5 @@
       <origin xyz="0 0 0" rpy=" 0 1.507 1.507"/>
       <geometry>
-        <cylinder length='0.05' radius='0.1'/>
+        <cylinder length='0.05' radius='0.05'/>
       </geometry>
     </collision>
@@ -98,10 +98,10 @@
       <origin xyz="0 0 0" rpy=" 0 1.507 1.507"/>
       <geometry>
-        <cylinder length='0.05' radius='0.1'/>
+        <cylinder length='0.05' radius='0.05'/>
       </geometry>
     </visual>
   </link>
 	<joint type="continuous" name="left_wheel_hinge">
-    <origin xyz="0 0.15 0" rpy="0 0 0"/>
+    <origin xyz="0 0.15 -0.05" rpy="0 0 0"/>
     <child link="left_wheel"/>
     <parent link="chassis"/>
@@ -111,6 +111,131 @@
   </joint>
 	<joint type="continuous" name="right_wheel_hinge">
-    <origin xyz="0 -0.15 0" rpy="0 0 0"/>
+    <origin xyz="0 -0.15 -0.05" rpy="0 0 0"/>
     <child link="right_wheel"/>
+    <parent link="chassis"/>
+    <axis xyz="0 1 0" rpy="0 0 0"/>
+    <limit effort="10000" velocity="1000"/>
+    <dynamics damping="1.0" friction="1.0"/>
+  </joint>
+  <!-- Optional -->
+  <link name='right_wheel_f'>
+    <inertial>
+      <mass value="5.0"/>
+      <origin xyz="0.0 0 0" rpy=" 0 0 0"/>
+      <inertia
+          ixx="0.1" ixy="0" ixz="0"
+          iyy="0.1" iyz="0"
+          izz="0.1"
+      />
+    </inertial>
+    <collision name='right_wheel_collision_f'>
+      <origin xyz="0 0 0" rpy=" 0 1.507 1.507"/>
+      <geometry>
+        <cylinder length='0.05' radius='0.05'/>
+      </geometry>
+    </collision>
+    <visual name='right_wheel_visual_f'>
+      <origin xyz="0 0 0" rpy=" 0 1.507 1.507"/>
+      <geometry>
+        <cylinder length='0.05' radius='0.05'/>
+      </geometry>
+    </visual>
+  </link>
+	<joint type="continuous" name="right_wheel_hinge_f">
+    <origin xyz="0.15 -0.15 -0.05" rpy="0 0 0"/>
+    <child link="right_wheel_f"/>
+    <parent link="chassis"/>
+    <axis xyz="0 1 0" rpy="0 0 0"/>
+    <limit effort="10000" velocity="1000"/>
+    <dynamics damping="1.0" friction="1.0"/>
+  </joint>
+  <link name='right_wheel_b'>
+    <inertial>
+      <mass value="5.0"/>
+      <origin xyz="0.0 0 0" rpy=" 0 0 0"/>
+      <inertia
+          ixx="0.1" ixy="0" ixz="0"
+          iyy="0.1" iyz="0"
+          izz="0.1"
+      />
+    </inertial>
+    <collision name='right_wheel_collision_b'>
+      <origin xyz="0 0 0" rpy=" 0 1.507 1.507"/>
+      <geometry>
+        <cylinder length='0.05' radius='0.05'/>
+      </geometry>
+    </collision>
+    <visual name='right_wheel_visual_b'>
+      <origin xyz="0 0 0" rpy=" 0 1.507 1.507"/>
+      <geometry>
+        <cylinder length='0.05' radius='0.05'/>
+      </geometry>
+    </visual>
+  </link>
+	<joint type="continuous" name="right_wheel_hinge_b">
+    <origin xyz="-0.15 -0.15 -0.05" rpy="0 0 0"/>
+    <child link="right_wheel_b"/>
+    <parent link="chassis"/>
+    <axis xyz="0 1 0" rpy="0 0 0"/>
+    <limit effort="10000" velocity="1000"/>
+    <dynamics damping="1.0" friction="1.0"/>
+  </joint>
+  <link name='left_wheel_f'>
+    <inertial>
+      <mass value="5.0"/>
+      <origin xyz="0.0 0 0" rpy=" 0 0 0"/>
+      <inertia
+          ixx="0.1" ixy="0" ixz="0"
+          iyy="0.1" iyz="0"
+          izz="0.1"
+      />
+    </inertial>
+    <collision name='left_wheel_collision_f'>
+      <origin xyz="0 0 0" rpy=" 0 1.507 1.507"/>
+      <geometry>
+        <cylinder length='0.05' radius='0.05'/>
+      </geometry>
+    </collision>
+    <visual name='left_wheel_visual_f'>
+      <origin xyz="0 0 0" rpy=" 0 1.507 1.507"/>
+      <geometry>
+        <cylinder length='0.05' radius='0.05'/>
+      </geometry>
+    </visual>
+  </link>
+  <joint type="continuous" name="left_wheel_hinge_f">
+    <origin xyz="0.15 0.15 -0.05" rpy="0 0 0"/>
+    <child link="left_wheel_f"/>
+    <parent link="chassis"/>
+    <axis xyz="0 1 0" rpy="0 0 0"/>
+    <limit effort="10000" velocity="1000"/>
+    <dynamics damping="1.0" friction="1.0"/>
+  </joint>
+  <link name='left_wheel_b'>
+    <inertial>
+      <mass value="5.0"/>
+      <origin xyz="0.0 0 0" rpy=" 0 0 0"/>
+      <inertia
+          ixx="0.1" ixy="0" ixz="0"
+          iyy="0.1" iyz="0"
+          izz="0.1"
+      />
+    </inertial>
+    <collision name='left_wheel_collision_b'>
+      <origin xyz="0 0 0" rpy=" 0 1.507 1.507"/>
+      <geometry>
+        <cylinder length='0.05' radius='0.05'/>
+      </geometry>
+    </collision>
+    <visual name='left_wheel_visual_b'>
+      <origin xyz="0 0 0" rpy=" 0 1.507 1.507"/>
+      <geometry>
+        <cylinder length='0.05' radius='0.05'/>
+      </geometry>
+    </visual>
+  </link>
+  <joint type="continuous" name="left_wheel_hinge_b">
+    <origin xyz="-0.15 0.15 -0.05" rpy="0 0 0"/>
+    <child link="left_wheel_b"/>
     <parent link="chassis"/>
     <axis xyz="0 1 0" rpy="0 0 0"/>
@@ -176,5 +301,5 @@
     <axis xyz="0 1 0" rpy="0 0 0"/>
   </joint>
-	<gazebo reference="left_wheel">
+  <gazebo reference="left_wheel">
     <material>Gazebo/Green</material>
 	</gazebo>

Commit message: Fix angles in urdf (1.507 rad instead of 1.5707)

File: Project 2/my_robot/urdf/my_robot.xacro (robot description, xacro)
@@ -67,5 +67,5 @@
     </inertial>
     <collision name='left_wheel_collision'>
-      <origin xyz="0 0 0" rpy=" 0 1.507 1.507"/>
+      <origin xyz="0 0 0" rpy=" 0 1.5707 1.5707"/>
       <geometry>
         <cylinder length='0.05' radius='0.05'/>
@@ -73,5 +73,5 @@
     </collision>
     <visual name='left_wheel_visual'>
-      <origin xyz="0 0 0" rpy=" 0 1.507 1.507"/>
+      <origin xyz="0 0 0" rpy=" 0 1.5707 1.5707"/>
       <geometry>
         <cylinder length='0.05' radius='0.05'/>
@@ -90,5 +90,5 @@
     </inertial>
     <collision name='right_wheel_collision'>
-      <origin xyz="0 0 0" rpy=" 0 1.507 1.507"/>
+      <origin xyz="0 0 0" rpy=" 0 1.5707 1.5707"/>
       <geometry>
         <cylinder length='0.05' radius='0.05'/>
@@ -96,5 +96,5 @@
     </collision>
     <visual name='right_wheel_visual'>
-      <origin xyz="0 0 0" rpy=" 0 1.507 1.507"/>
+      <origin xyz="0 0 0" rpy=" 0 1.5707 1.5707"/>
       <geometry>
         <cylinder length='0.05' radius='0.05'/>
@@ -130,5 +130,5 @@
     </inertial>
     <collision name='right_wheel_collision_f'>
-      <origin xyz="0 0 0" rpy=" 0 1.507 1.507"/>
+      <origin xyz="0 0 0" rpy=" 0 1.5707 1.5707"/>
       <geometry>
         <cylinder length='0.05' radius='0.05'/>
@@ -136,5 +136,5 @@
     </collision>
     <visual name='right_wheel_visual_f'>
-      <origin xyz="0 0 0" rpy=" 0 1.507 1.507"/>
+      <origin xyz="0 0 0" rpy=" 0 1.5707 1.5707"/>
       <geometry>
         <cylinder length='0.05' radius='0.05'/>
@@ -161,5 +161,5 @@
     </inertial>
     <collision name='right_wheel_collision_b'>
-      <origin xyz="0 0 0" rpy=" 0 1.507 1.507"/>
+      <origin xyz="0 0 0" rpy=" 0 1.5707 1.5707"/>
       <geometry>
         <cylinder length='0.05' radius='0.05'/>
@@ -167,5 +167,5 @@
     </collision>
     <visual name='right_wheel_visual_b'>
-      <origin xyz="0 0 0" rpy=" 0 1.507 1.507"/>
+      <origin xyz="0 0 0" rpy=" 0 1.5707 1.5707"/>
       <geometry>
         <cylinder length='0.05' radius='0.05'/>
@@ -192,5 +192,5 @@
     </inertial>
     <collision name='left_wheel_collision_f'>
-      <origin xyz="0 0 0" rpy=" 0 1.507 1.507"/>
+      <origin xyz="0 0 0" rpy=" 0 1.5707 1.5707"/>
       <geometry>
         <cylinder length='0.05' radius='0.05'/>
@@ -198,5 +198,5 @@
     </collision>
     <visual name='left_wheel_visual_f'>
-      <origin xyz="0 0 0" rpy=" 0 1.507 1.507"/>
+      <origin xyz="0 0 0" rpy=" 0 1.5707 1.5707"/>
       <geometry>
         <cylinder length='0.05' radius='0.05'/>
@@ -223,5 +223,5 @@
     </inertial>
     <collision name='left_wheel_collision_b'>
-      <origin xyz="0 0 0" rpy=" 0 1.507 1.507"/>
+      <origin xyz="0 0 0" rpy=" 0 1.5707 1.5707"/>
       <geometry>
         <cylinder length='0.05' radius='0.05'/>
@@ -229,5 +229,5 @@
     </collision>
     <visual name='left_wheel_visual_b'>
-      <origin xyz="0 0 0" rpy=" 0 1.507 1.507"/>
+      <origin xyz="0 0 0" rpy=" 0 1.5707 1.5707"/>
       <geometry>
         <cylinder length='0.05' radius='0.05'/>
