Commit message: fix: Make the whole project and AMCL runnable
- Change amcl.launch and add parameters to improve MC algorithm quality (still not perfect so further tuning is needed)
- Tune parameters .yaml files to remove warning messages when running
- Change RViz config file to load correct items
- Remove extra robot wheels to grant better speed and performances

File: Project_3/my_robot/urdf/my_robot.xacro (robot description, xacro)
@@ -119,5 +119,5 @@
   </joint>
   <!-- Optional -->
-  <link name='right_wheel_f'>
+  <!-- <link name='right_wheel_f'>
     <inertial>
       <mass value="5.0"/>
@@ -242,5 +242,5 @@
     <limit effort="10000" velocity="1000"/>
     <dynamics damping="1.0" friction="1.0"/>
-  </joint>
+  </joint> -->
 	<link name='camera'>
 		<inertial>
